File: A600KB.kicad_pcb (KiCad board)
At the start: 2 copper layers, 324 x 124.5 mm, 81 parts, among them J1 32 FFC

Commit message: update kicad version
Other:
- net class Default removed

Commit message: Revise PCB to fix swapped keys
Parts:
- moved MX79 51.4 mm to (239.9, 136.2)
- moved MX63 51.4 mm to (287.7, 117.1)
Connections:
- J1 pad 31: Net-(J1-Pad31) -> unconnected-(J1-Pad31)
- J1 pad 32: Net-(J1-Pad32) -> unconnected-(J1-Pad32)
Routing:
- net /26: track 226.4 -> 152.0 mm
- net /3: track 431.0 -> 361.8 mm
- net /5: track 478.8 -> 418.7 mm, vias 2 -> 0
- net /2: track 390.3 -> 332.4 mm, vias 1 -> 0
- net /23: track 188.4 -> 144.3 mm
- net /7: track 469.1 -> 441.5 mm, vias 2 -> 0
- net /15: track 279.1 -> 253.6 mm, vias 4 -> 2
- net /21: track 129.6 -> 104.4 mm
- net /29: track 362.5 -> 343.4 mm, vias 1 -> 0
- net /4: track 142.8 -> 161.0 mm, vias 1 -> 2
- net /6: track 233.8 -> 225.1 mm
- net /28: track 228.4 -> 221.9 mm
- net /10: track 168.5 -> 174.6 mm
- net /27: track 286.7 -> 292.1 mm
- net /22: track 89.4 -> 85.4 mm
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Other:
- board text added: "A600 KB r2 - aeberbach - grayunicorn.com - May ‘22"
- board text removed: "A600 KB r1 - aeberbach - grayunicorn.com - Nov ‘19"
